Commit message: fix: Isaac Sim 5.1.0 full compatibility - state machine PASS

File: assets/robots/rm75b/rm75b_local.urdf (robot description, URDF)
Before this commit: robot RM75-B_with_Gripper, 15 links, 14 joints
Links:
- link Left_1_Link: geometry collision mesh filename=../gripper/meshes/Left_1_Link.STL; visual mesh filename=../gripper/meshes/Left_1_Link.STL
- link Left_2_Link: geometry collision mesh filename=../gripper/meshes/Left_2_Link.STL; visual mesh filename=../gripper/meshes/Left_2_Link.STL
- link Left_Support_Link: geometry collision mesh filename=../gripper/meshes/Left_Support_Link.STL; visual mesh filename=../gripper/meshes/Left_Support_Link.STL
- link Right_1_Link: geometry collision mesh filename=../gripper/meshes/Right_1_Link.STL; visual mesh filename=../gripper/meshes/Right_1_Link.STL
- link Right_2_Link: geometry collision mesh filename=../gripper/meshes/Right_2_Link.STL; visual mesh filename=../gripper/meshes/Right_2_Link.STL
- link Right_Support_Link: geometry collision mesh filename=../gripper/meshes/Right_Support_Link.STL; visual mesh filename=../gripper/meshes/Right_Support_Link.STL
- link gripper_base_link: geometry collision mesh filename=../gripper/meshes/base_link.STL; visual mesh filename=../gripper/meshes/base_link.STL

Commit message: Add RMPFlow to robotic arm

File: assets/robots/rm75b/rm75b_local.urdf (robot description, URDF)
Before this commit: robot RM75-B_with_Gripper, 15 links, 14 joints
Joints:
- joint Left_1_Joint: limit lower=-0.91 upper=0 effort=10 velocity=10 -> lower=-0.5 upper=0.5 effort=5 velocity=1.0
- joint Left_2_Joint: limit lower=0 upper=0 effort=0 velocity=0 -> lower=-0.5 upper=0.5 effort=5 velocity=1.0
- joint Left_Support_Joint: type revolute -> fixed
- joint Right_1_Joint: limit lower=0 upper=0 effort=0 velocity=0 -> lower=-0.5 upper=0.5 effort=5 velocity=1.0
- joint Right_2_Joint: limit lower=0 upper=0 effort=0 velocity=0 -> lower=-0.5 upper=0.5 effort=5 velocity=1.0
- joint Right_Support_Joint: type revolute -> fixed

Commit message: change rm75b urdf

File: assets/robots/rm75b/rm75b_local.urdf (robot description, URDF)
Before this commit: robot RM75-B_with_Gripper, 15 links, 14 joints
Joints:
- joint Left_2_Joint: axis 0 0 -1 -> (none); limit lower=-0.5 upper=0.5 effort=5 velocity=1.0 -> (none); mimic joint=Left_1_Joint multiplier=1 offset=0 -> (none); type revolute -> fixed
- joint Left_Support_Joint: axis 0 0 -1 -> (none); limit lower=0 upper=0 effort=0 velocity=0 -> (none); mimic joint=Left_1_Joint multiplier=-1 offset=0 -> (none)
- joint Right_1_Joint: axis 0 0 1 -> (none); limit lower=-0.5 upper=0.5 effort=5 velocity=1.0 -> (none); mimic joint=Left_1_Joint multiplier=-1 offset=0 -> (none); type revolute -> fixed
- joint Right_2_Joint: axis 0 0 1 -> (none); limit lower=-0.5 upper=0.5 effort=5 velocity=1.0 -> (none); mimic joint=Left_1_Joint multiplier=-1 offset=0 -> (none); type revolute -> fixed
- joint Right_Support_Joint: axis 0 0 -1 -> (none); limit lower=0 upper=0 effort=0 velocity=0 -> (none); mimic joint=Left_1_Joint multiplier=-1 offset=0 -> (none)
